File: GTB.sch (KiCad schematic (older format))
At the start: 1 part

Commit message: Finished Schematic
Parts:
- added BT1: CR2032, ~, symbol BATTERY
- added C1: 1U, ~, symbol C
- added D1: LED, ~, symbol LED
- added R1: 470K, ~, symbol R
- added R2: 1K, ~, symbol R
- added VR1: LDR, ~, symbol VR
- gave numbers to parts that had none: 1
Connections:
- net GND: now reaches U1.1 (GND)
- net GND: now also BT1.2 (-), C1.2, D1.2 (K)
- net at U1.2 (TRIG): now also U1.6 (THR), C1.1, R1.2
- net at U1.3 (OUT): now also R2.1
- net VCC: now reaches U1.4 (~RESET)
- net VCC: now also U1.8 (VCC), BT1.1 (+), VR1.1
- net at U1.7 (DIS): now also R1.1, VR1.2
- new net: D1.1 (A), R2.2
Changed lines of the file:
@@
-EESchema Schematic File Version 2  date 10/1/2013 12:22:22 AM
+EESchema Schematic File Version 2  date 10/2/2013 12:47:39 AM
 LIBS:power
 LIBS:device
@@
 Sheet 1 1
 Title ""
-Date "1 oct 2013"
+Date "2 oct 2013"
 Rev ""
 Comp ""
@@
 $EndDescr
 $Comp
-L 7555 U?
+L 7555 U1
 U 1 1 524A4F04
 P 4450 4100
-F 0 "U?" H 5150 3700 60  0000 C CNN
+F 0 "U1" H 5150 3700 60  0000 C CNN
 F 1 "7555" H 4600 4350 60  0000 C CNN
 F 2 "" H 4400 3900 60  0000 C CNN
@@
 	1    0    0    -1
 $EndComp
+$Comp
+L C C1
+U 1 1 524BA208
+P 2750 4550
+F 0 "C1" H 2750 4650 40  0000 L CNN
+F 1 "1U" H 2756 4465 40  0000 L CNN
+F 2 "~" H 2788 4400 30  0000 C CNN
+F 3 "~" H 2750 4550 60  0000 C CNN
+	1    2750 4550
+	1    0    0    -1
+$EndComp
+$Comp
+L R R1
+U 1 1 524BA21F
+P 2750 3950
+F 0 "R1" V 2830 3950 40  0000 C CNN
+F 1 "470K" V 2757 3951 40  0000 C CNN
+F 2 "~" V 2680 3950 30  0000 C CNN
+F 3 "~" H 2750 3950 30  0000 C CNN
+	1    2750 3950
+	1    0    0    -1
+$EndComp
+$Comp
+L VR VR1
+U 1 1 524BA23A
+P 2750 3250
+F 0 "VR1" V 2810 3204 40  0000 C TNN
+F 1 "LDR" V 2750 3250 40  0000 C CNN
+F 2 "~" H 2750 3250 60  0000 C CNN
+F 3 "~" H 2750 3250 60  0000 C CNN
+	1    2750 3250
+	1    0    0    -1
+$EndComp
+$Comp
+L R R2
+U 1 1 524BA251
+P 5850 4200
+F 0 "R2" V 5930 4200 40  0000 C CNN
+F 1 "1K" V 5857 4201 40  0000 C CNN
+F 2 "~" V 5780 4200 30  0000 C CNN
+F 3 "~" H 5850 4200 30  0000 C CNN
+	1    5850 4200
+	1    0    0    -1
+$EndComp
+$Comp
+L LED D1
+U 1 1 524BA266
+P 5850 4950
+F 0 "D1" H 5850 5050 50  0000 C CNN
+F 1 "LED" H 5850 4850 50  0000 C CNN
+F 2 "~" H 5850 4950 60  0000 C CNN
+F 3 "~" H 5850 4950 60  0000 C CNN
+	1    5850 4950
+	0    1    1    0
+$EndComp
+Wire Wire Line
+	2750 3500 2750 3700
+Wire Wire Line
+	3600 3550 2750 3550
+Connection ~ 2750 3550
+Wire Wire Line
+	2750 4200 2750 4350
+Wire Wire Line
+	3600 4100 3250 4100
+Wire Wire Line
+	3250 3800 3250 4300
+Wire Wire Line
+	3250 4300 2750 4300
+Connection ~ 2750 4300
+Wire Wire Line
+	3250 3800 3600 3800
+Connection ~ 3250 4100
+Wire Wire Line
+	4350 4700 4350 5300
+Wire Wire Line
+	2750 5300 5850 5300
+Wire Wire Line
+	2750 4750 2750 5950
+Wire Wire Line
+	5850 4750 5850 4450
+Wire Wire Line
+	5850 3950 5850 3900
+Wire Wire Line
+	5850 3900 5500 3900
+Wire Wire Line
+	4350 3050 4350 2700
+Wire Wire Line
+	2750 2700 4750 2700
+Wire Wire Line
+	4750 2700 4750 3050
+Wire Wire Line
+	5850 5300 5850 5150
+Connection ~ 4350 5300
+$Comp
+L VCC #PWR01
+U 1 1 524BA329
+P 2750 2150
+F 0 "#PWR01" H 2750 2250 30  0001 C CNN
+F 1 "VCC" H 2750 2250 30  0000 C CNN
+F 2 "~" H 2750 2150 60  0000 C CNN
+F 3 "~" H 2750 2150 60  0000 C CNN
+	1    2750 2150
+	1    0    0    -1
+$EndComp
+Wire Wire Line
+	2750 2150 2750 3000
+Connection ~ 2750 2700
+Connection ~ 4350 2700
+$Comp
+L GND #PWR02
+U 1 1 524BA37E
+P 2750 5950
+F 0 "#PWR02" H 2750 5950 30  0001 C CNN
+F 1 "GND" H 2750 5880 30  0001 C CNN
+F 2 "~" H 2750 5950 60  0000 C CNN
+F 3 "~" H 2750 5950 60  0000 C CNN
+	1    2750 5950
+	1    0    0    -1
+$EndComp
+Connection ~ 2750 5300
+$Comp
+L BATTERY BT1
+U 1 1 524BA3C2
+P 1050 4500
+F 0 "BT1" H 1050 4700 50  0000 C CNN
+F 1 "CR2032" H 1050 4310 50  0000 C CNN
+F 2 "~" H 1050 4500 60  0000 C CNN
+F 3 "~" H 1050 4500 60  0000 C CNN
+	1    1050 4500
+	0    1    1    0
+$EndComp
+$Comp
+L VCC #PWR03
+U 1 1 524BA3CF
+P 1050 3850
+F 0 "#PWR03" H 1050 3950 30  0001 C CNN
+F 1 "VCC" H 1050 3950 30  0000 C CNN
+F 2 "~" H 1050 3850 60  0000 C CNN
+F 3 "~" H 1050 3850 60  0000 C CNN
+	1    1050 3850
+	1    0    0    -1
+$EndComp
+$Comp
+L GND #PWR04
+U 1 1 524BA3D5
+P 1050 5050
+F 0 "#PWR04" H 1050 5050 30  0001 C CNN
+F 1 "GND" H 1050 4980 30  0001 C CNN
+F 2 "~" H 1050 5050 60  0000 C CNN
+F 3 "~" H 1050 5050 60  0000 C CNN
+	1    1050 5050
+	1    0    0    -1
+$EndComp
+Wire Wire Line
+	1050 5050 1050 4800
+Wire Wire Line
+	1050 4200 1050 3850
 $EndSCHEMATC
