File: GTB.kicad_pcb (KiCad board)
At the start: 2 copper layers, 0 parts

Commit message: Imported Footprints To Layout and Added CR2032 Footprint
Parts:
- added BT1: CR2032, CR2032, F.Cu at (43.4, 31.0)
- added C1: 1U, SM1206, F.Cu at (13.1, 1.02)
- added D1: LED, LED-1206, F.Cu at (14.5, 8.64)
- added R1: 470K, SM1206, F.Cu at (2.79, 8.76)
- added R2: 1K, SM1206, F.Cu at (8.76, 8.76)
- added U1: 7555, SO8N, F.Cu at (2.54, 3.56)
- added VR1: LDR, R1, F.Cu at (10.9, -3.94)

Commit message: Board Layout of the GTB 1 Sq In PCB
Parts:
- BT1: moved to B.Cu
- moved VR1 236.4 mm to (194.3, 145.2), turned to 90 degrees
- moved U1 235.2 mm to (183.1, 154.2), turned to 270 degrees
- moved C1 233.7 mm to (185.0, 159.3)
- moved D1 229.3 mm to (183.0, 164.1)
- moved R1 228.4 mm to (183.5, 148.5), turned to 180 degrees
- moved R2 224.7 mm to (176.1, 158.6), turned to 270 degrees
- moved BT1 184.4 mm to (183.3, 151.3), turned to 180 degrees
Routing:
- net N-000007: track 0.00 -> 19.4 mm
- net N-000005: track 0.00 -> 17.9 mm
- net GND: track 0.00 -> 12.4 mm, vias 0 -> 2
- net N-000002: track 0.00 -> 8.43 mm
- net N-000003: track 0.00 -> 5.45 mm
- added copper zone on B.Cu, net GND
- added copper zone on F.Cu, net VCC
Other:
- board outline added: 25.4 x 25.4 mm
- board text added: "CG"
- board text added: "Getting To Blinky"
